File: Headlights_Driver/Headlights_Driver.kicad_pcb (KiCad board)
At the start: 4 copper layers, 45.2 x 35.6 mm, 62 parts, among them J1 VS, J2 GND, J3 SWD, J4 VDD, J5 TX, J6 RX, J7 Vdrive, J8 LED+, J9 LED-, Q1 BSC190N12NS3G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

Commit message: ...
Other:
- board text added: "PCB3D_BR_HEADLIGHTSV2"
- board text added: "PCB3D_TL_HEADLIGHTSV2"
Changed lines of the file:
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@@
     (effects (font (size 1 1) (thickness 0.15)) (justify left))
+  )
+  (gr_text "PCB3D_BR_HEADLIGHTSV2" (at 168.656 95.25) (layer "F.Fab")
+    (effects (font (size 1 1) (thickness 0.15)) (justify left bottom))
+  )
+  (gr_text "PCB3D_TL_HEADLIGHTSV2" (at 123.444 59.69) (layer "F.Fab")
+    (effects (font (size 1 1) (thickness 0.15)) (justify left bottom))
   )
   (dimension (type aligned) (layer "Dwgs.User")
